File: Pedal_pcb/Pedal_pcb.kicad_pcb (KiCad board)
At the start: 2 copper layers, 40.5 x 48.5 mm, 18 parts, among them U1 TL082

Commit message: better pcb design
Parts:
- moved C6 3.64 mm to (129.0, 44.6)
- moved C7 3.64 mm to (129.0, 51.1)
- moved C3 3.64 mm to (129.0, 38.0)
- moved R3 1.98 mm to (139.4, 54.0)
- moved D2 1.00 mm to (125.2, 62.0)
- moved U1 1.00 mm to (155.4, 65.8)
- moved gain1 1.00 mm to (127.8, 31.0)
- moved tone1 1.00 mm to (141.7, 31.0)
- moved volume1 1.00 mm to (155.6, 31.0)
- moved C1 0.99 mm to (161.0, 46.5)
- moved C2 0.99 mm to (161.0, 35.0)
- moved C4 0.99 mm to (161.0, 40.5)
- moved C5 0.99 mm to (161.0, 52.5)
- moved D1 0.99 mm to (125.2, 58.5)
- moved R1 0.99 mm to (139.4, 35.5)
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Routing:
- net Net-(D1-A): track 103.2 -> 107.5 mm
- net Net-(C3-Pad1): track 28.0 -> 31.2 mm
- net GND: track 56.7 -> 54.1 mm
- net Net-(C6-Pad1): track 32.1 -> 29.5 mm
- net Net-(D1-K): track 102.6 -> 101.4 mm
- net Net-(BT1-+): track 28.2 -> 27.2 mm
Other:
- board size 40.5 x 48.5 mm -> 41.9 x 49.5 mm
- board text added: "Made in italy by italians"
- board text added: "R1"
- board text added: "R2"
- board text added: "R3"
- board text added: "R4"
- board text added: "R5"
- board text removed: "Made in italy by one italian"

Commit message: the pcb is done
Parts:
- added Battery1: Conn_01x02, TestPoint:TestPoint_2Pads_Pitch2.54mm_Drill0.8mm, F.Cu at (141.6, 62.2)
- added Input1: Conn_01x02, TestPoint:TestPoint_2Pads_Pitch2.54mm_Drill0.8mm, F.Cu at (158.1, 42.5)
- added Output1: Conn_01x02, TestPoint:TestPoint_2Pads_Pitch2.54mm_Drill0.8mm, F.Cu at (126.4, 42.5)
- moved R2 2.31 mm to (141.0, 57.8)
- moved R3 1.27 mm to (139.4, 52.7)
Routing:
- net Net-(Output1-Pin_2): track 0.00 -> 44.4 mm
- net Net-(Input1-Pin_1): track 0.00 -> 38.8 mm
- net GND: track 54.1 -> 83.7 mm
- net Net-(Battery1-Pin_1): track 27.2 -> 44.4 mm
- net Net-(C5-Pad1): track 14.3 -> 12.1 mm
- net Net-(D1-K): track 101.4 -> 102.9 mm
- net Net-(U1A-+): track 39.7 -> 41.0 mm
- net Net-(D1-A): track 107.5 -> 108.5 mm

Commit message: final pcb
Parts:
- moved Output1 1.27 mm to (125.1, 42.5)
Routing:
- net GND: track 83.7 -> 84.2 mm
Other:
- board size 41.9 x 49.5 mm -> 47 x 49.5 mm
Changed lines of the file:
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@@
 	(footprint "TestPoint:TestPoint_2Pads_Pitch2.54mm_Drill0.8mm"
 		(layer "F.Cu")
-		(at 126.365 42.525 90)
+		(at 125.095 42.525 90)
 		(descr "Test point with 2 pins, pitch 2.54mm, drill diameter 0.8mm")
 		(tags "CONN DEV")
@@
 	)
 	(gr_rect
-		(start 123.19 17.78)
-		(end 165.1 67.31)
+		(start 120.65 17.78)
+		(end 167.64 67.31)
+		(stroke
+			(width 0.05)
+			(type default)
+		)
+		(fill no)
+		(layer "Edge.Cuts")
+	)
+	(gr_circle
+		(center 121.92 19.05)
+		(end 121.285 18.415)
+		(stroke
+			(width 0.05)
+			(type default)
+		)
+		(fill no)
+		(layer "Edge.Cuts")
+	)
+	(gr_circle
+		(center 121.92 66.04)
+		(end 121.285 66.675)
+		(stroke
+			(width 0.05)
+			(type default)
+		)
+		(fill no)
+		(layer "Edge.Cuts")
+	)
+	(gr_circle
+		(center 166.37 19.05)
+		(end 167.005 18.415)
+		(stroke
+			(width 0.05)
+			(type default)
+		)
+		(fill no)
+		(layer "Edge.Cuts")
+	)
+	(gr_circle
+		(center 166.37 66.04)
+		(end 167.005 66.675)
 		(stroke
 			(width 0.05)
@@
 	)
 	(segment
+		(start 126.834315 28.81)
+		(end 125.33 30.314314)
+		(width 0.2)
+		(layer "F.Cu")
+		(net "Net-(Output1-Pin_2)")
+	)
+	(segment
+		(start 158.07 30.995)
+		(end 155.885 28.81)
+		(width 0.2)
+		(layer "F.Cu")
+		(net "Net-(Output1-Pin_2)")
+	)
+	(segment
+		(start 125.33 30.314314)
+		(end 125.33 39.75)
+		(width 0.2)
+		(layer "F.Cu")
+		(net "Net-(Output1-Pin_2)")
+	)
+	(segment
+		(start 125.33 39.75)
+		(end 125.095 39.985)
+		(width 0.2)
+		(layer "F.Cu")
+		(net "Net-(Output1-Pin_2)")
+	)
+	(segment
+		(start 155.885 28.81)
+		(end 126.834315 28.81)
+		(width 0.2)
+		(layer "F.Cu")
+		(net "Net-(Output1-Pin_2)")
+	)
+	(segment
 		(start 161 34.995)
 		(end 161 37.995)
@@
 	)
 	(segment
+		(start 125.095 42.544744)
+		(end 125.095 42.525)
+		(width 0.2)
+		(layer "B.Cu")
+		(net "GND")
+	)
+	(segment
 		(start 158.815 39.285)
 		(end 162.29 39.285)
@@
 	)
 	(segment
-		(start 126.365 43.814744)
-		(end 128.240144 45.689888)
-		(width 0.2)
-		(layer "B.Cu")
-		(net "GND")
-	)
-	(segment
 		(start 139.42 50.52)
 		(end 139.42 47.995)
@@
 	)
 	(segment
-		(start 126.365 42.525)
-		(end 126.365 43.814744)
-		(width 0.2)
-		(layer "B.Cu")
-		(net "GND")
-	)
-	(segment
 		(start 134.169776 47.995)
 		(end 131.024888 51.139888)
@@
 	)
 	(segment
+		(start 128.240144 45.689888)
+		(end 125.095 42.544744)
+		(width 0.2)
+		(layer "B.Cu")
+		(net "GND")
+	)
+	(segment
 		(start 144.165 55.265)
 		(end 139.42 50.52)
@@
 	)
 	(segment
+		(start 133.53 43.995)
+		(end 129.024888 48.500112)
+		(width 0.2)
+		(layer "B.Cu")
+		(net "Net-(Battery1-Pin_1)")
+	)
+	(segment
+		(start 141.625 62.23)
+		(end 140.115 62.23)
+		(width 0.2)
+		(layer "B.Cu")
+		(net "Net-(Battery1-Pin_1)")
+	)
+	(segment
+		(start 140.115 62.23)
+		(end 129.024888 51.139888)
+		(width 0.2)
+		(layer "B.Cu")
+		(net "Net-(Battery1-Pin_1)")
+	)
+	(segment
+		(start 149 43.995)
+		(end 133.53 43.995)
+		(width 0.2)
+		(layer "B.Cu")
+		(net "Net-(Battery1-Pin_1)")
+	)
+	(segment
+		(start 149.58 41.495)
+		(end 149.58 43.415)
+		(width 0.2)
+		(layer "B.Cu")
+		(net "Net-(Battery1-Pin_1)")
+	)
+	(segment
+		(start 129.024888 48.500112)
+		(end 129.024888 51.139888)
+		(width 0.2)
+		(layer "B.Cu")
+		(net "Net-(Battery1-Pin_1)")
+	)
+	(segment
+		(start 149.58 43.415)
+		(end 149 43.995)
+		(width 0.2)
+		(layer "B.Cu")
+		(net "Net-(Battery1-Pin_1)")
+	)
+	(segment
+		(start 137.795 50.8)
+		(end 137.16 51.435)
+		(width 0.2)
+		(layer "F.Cu")
+		(net "Net-(Input1-Pin_1)")
+	)
+	(segment
+		(start 158.115 42.525)
+		(end 158.115 47.625)
+		(width 0.2)
+		(layer "F.Cu")
+		(net "Net-(Input1-Pin_1)")
+	)
+	(segment
+		(start 140.97 50.8)
+		(end 137.795 50.8)
+		(width 0.2)
+		(layer "F.Cu")
+		(net "Net-(Input1-Pin_1)")
+	)
+	(segment
+		(start 158.115 47.625)
+		(end 151.065 54.675)
+		(width 0.2)
+		(layer "F.Cu")
+		(net "Net-(Input1-Pin_1)")
+	)
+	(segment
+		(start 137.16 53.975)
+		(end 140.97 57.785)
+		(width 0.2)
+		(layer "F.Cu")
+		(net "Net-(Input1-Pin_1)")
+	)
+	(segment
+		(start 144.844999 54.675)
+		(end 140.97 50.8)
+		(width 0.2)
+		(layer "F.Cu")
+		(net "Net-(Input1-Pin_1)")
+	)
+	(segment
+		(start 151.065 54.675)
+		(end 144.844999 54.675)
+		(width 0.2)
+		(layer "F.Cu")
+		(net "Net-(Input1-Pin_1)")
+	)
+	(segment
+		(start 137.16 51.435)
+		(end 137.16 53.975)
+		(width 0.2)
+		(layer "F.Cu")
+		(net "Net-(Input1-Pin_1)")
+	)
+	(segment
 		(start 161 52.495)
 		(end 156.42 52.495)
@@
 		(net "Net-(C2-Pad2)")
 	)
-	(segment
-		(start 133.53 43.995)
-		(end 129.024888 48.500112)
-		(width 0.2)
-		(layer "B.Cu")
-		(net "Net-(Battery1-Pin_1)")
-	)
-	(segment
-		(start 141.625 62.23)
-		(end 140.115 62.23)
-		(width 0.2)
-		(layer "B.Cu")
-		(net "Net-(Battery1-Pin_1)")
-	)
-	(segment
-		(start 140.115 62.23)
-		(end 129.024888 51.139888)
-		(width 0.2)
-		(layer "B.Cu")
-		(net "Net-(Battery1-Pin_1)")
-	)
-	(segment
-		(start 149 43.995)
-		(end 133.53 43.995)
-		(width 0.2)
-		(layer "B.Cu")
-		(net "Net-(Battery1-Pin_1)")
-	)
-	(segment
-		(start 149.58 41.495)
-		(end 149.58 43.415)
-		(width 0.2)
-		(layer "B.Cu")
-		(net "Net-(Battery1-Pin_1)")
-	)
-	(segment
-		(start 129.024888 48.500112)
-		(end 129.024888 51.139888)
-		(width 0.2)
-		(layer "B.Cu")
-		(net "Net-(Battery1-Pin_1)")
-	)
-	(segment
-		(start 149.58 43.415)
-		(end 149 43.995)
-		(width 0.2)
-		(layer "B.Cu")
-		(net "Net-(Battery1-Pin_1)")
-	)
-	(segment
-		(start 137.795 50.8)
-		(end 137.16 51.435)
-		(width 0.2)
-		(layer "F.Cu")
-		(net "Net-(Input1-Pin_1)")
-	)
-	(segment
-		(start 158.115 42.525)
-		(end 158.115 47.625)
-		(width 0.2)
-		(layer "F.Cu")
-		(net "Net-(Input1-Pin_1)")
-	)
-	(segment
-		(start 140.97 50.8)
-		(end 137.795 50.8)
-		(width 0.2)
-		(layer "F.Cu")
-		(net "Net-(Input1-Pin_1)")
-	)
-	(segment
-		(start 158.115 47.625)
-		(end 151.065 54.675)
-		(width 0.2)
-		(layer "F.Cu")
-		(net "Net-(Input1-Pin_1)")
-	)
-	(segment
-		(start 137.16 53.975)
-		(end 140.97 57.785)
-		(width 0.2)
-		(layer "F.Cu")
-		(net "Net-(Input1-Pin_1)")
-	)
-	(segment
-		(start 144.844999 54.675)
-		(end 140.97 50.8)
-		(width 0.2)
-		(layer "F.Cu")
-		(net "Net-(Input1-Pin_1)")
-	)
-	(segment
-		(start 151.065 54.675)
-		(end 144.844999 54.675)
-		(width 0.2)
-		(layer "F.Cu")
-		(net "Net-(Input1-Pin_1)")
-	)
-	(segment
-		(start 137.16 51.435)
-		(end 137.16 53.975)
-		(width 0.2)
-		(layer "F.Cu")
-		(net "Net-(Input1-Pin_1)")
-	)
-	(segment
-		(start 155.885 28.81)
-		(end 158.07 30.995)
-		(width 0.2)
-		(layer "F.Cu")
-		(net "Net-(Output1-Pin_2)")
-	)
-	(segment
-		(start 125.33 38.95)
-		(end 125.33 30.314314)
-		(width 0.2)
-		(layer "F.Cu")
-		(net "Net-(Output1-Pin_2)")
-	)
-	(segment
-		(start 126.365 39.985)
-		(end 125.33 38.95)
-		(width 0.2)
-		(layer "F.Cu")
-		(net "Net-(Output1-Pin_2)")
-	)
-	(segment
-		(start 126.834315 28.81)
-		(end 155.885 28.81)
-		(width 0.2)
-		(layer "F.Cu")
-		(net "Net-(Output1-Pin_2)")
-	)
-	(segment
-		(start 125.33 30.314314)
-		(end 126.834315 28.81)
-		(width 0.2)
-		(layer "F.Cu")
-		(net "Net-(Output1-Pin_2)")
-	)
 	(embedded_fonts no)

Commit message: pcb
Parts:
- added SW1: SW_Nidec_CAS-120A1, Connector_PinHeader_2.54mm:PinHeader_1x03_P2.54mm_Vertical, F.Cu at (126.5, 60.7)
- moved Battery1 28.8 mm to (116.8, 47.6), turned to 90 degrees
- moved R2 22.2 mm to (118.9, 55.4)
- moved Input1 20.4 mm to (137.8, 40.6)
- moved C3 20.4 mm to (108.7, 36.1)
- moved C6 20.4 mm to (108.7, 42.7)
- moved C7 20.4 mm to (108.7, 49.2)
- moved C1 20.4 mm to (140.7, 44.6)
- moved C2 20.4 mm to (140.7, 33.1)
- moved C4 20.4 mm to (140.7, 38.6)
- moved C5 20.4 mm to (140.7, 50.6)
- moved D1 20.4 mm to (104.9, 56.6)
- moved D2 20.4 mm to (104.9, 60.1)
- moved Output1 20.4 mm to (104.8, 40.6)
- moved R1 20.4 mm to (119.1, 33.6)
- moved R3 20.4 mm to (119.1, 50.8)
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Connections:
- R2 pad 1: Net-(Input1-Pin_1) -> Net-(SW1-A)
Routing:
- net Net-(Output1-Pin_2): track 44.0 -> 82.1 mm
- net GND: track 84.2 -> 72.3 mm
- net Net-(Battery1-Pin_1): track 44.4 -> 37.9 mm
- net Net-(SW1-A): track 0.00 -> 6.39 mm
- net Net-(D1-A): track 108.5 -> 102.7 mm
- net Net-(Input1-Pin_1): track 38.8 -> 43.1 mm
- net Net-(U1A-+): track 41.0 -> 44.0 mm
- net Net-(C5-Pad1): track 12.1 -> 14.4 mm
- net Net-(C4-Pad1): track 20.7 -> 22.4 mm
Other:
- board text removed: "Made in italy by italians"

Commit message: pcb better
Parts:
- moved D1 0.96 mm to (104.9, 55.6)
Connections:
- C5 pad 2: Net-(U1A-+) -> Net-(Battery1-Pin_1)
- C7 pad 1: Net-(Battery1-Pin_1) -> Net-(SW1-A)
- Input1 pad 1: Net-(Input1-Pin_1) -> Net-(Battery1-Pin_1)
- R3 pad 1: Net-(U1A-+) -> Net-(Battery1-Pin_1)
- R4 pad 2: Net-(Battery1-Pin_1) -> Net-(SW1-A)
- SW1 pad 2: Net-(Input1-Pin_1) -> Net-(Battery1-Pin_1)
- U1 pad 3: Net-(U1A-+) -> Net-(Battery1-Pin_1)
Routing:
- net Net-(U1A-+): track 44.0 -> 0.00 mm
- net Net-(Input1-Pin_1): track 43.1 -> 0.00 mm
- net Net-(SW1-A): track 6.39 -> 46.1 mm
- net Net-(Battery1-Pin_1): track 37.9 -> 66.6 mm
- net Net-(Output1-Pin_2): track 82.1 -> 87.3 mm
- net Net-(D1-K): track 103.3 -> 104.0 mm
Other:
- board text added: "pedal in bypass"
