File: Pedal_pcb/Pedal_pcb.kicad_sch (KiCad schematic)
At the start: 22 parts, among them J1 AudioJack2, J2 AudioJack2, SW1 SW_SPDT, U1 TL082

Commit message: complete pcb
Parts:
- removed SW1: SW_SPDT, symbol Switch:SW_SPDT
- BT1: footprint Package_DFN_QFN:Texas_R-PUQFN-N10 -> (none)
- U1: footprint Package_DFN_QFN:Texas_DSQ0010A_WSON-10-1EP_2x2mm_P0.4mm_EP0.9x1.5mm -> Package_DIP:DIP-8_W7.62mm
- renumbered gain to gain1, tone to tone1, volume to volume1
Connections:
- net at BT1.1 (+): now also C7.1, R4.2
Changed lines of the file:
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@@
+	)
+	(junction
+		(at 121.92 50.8)
+		(diameter 0)
+		(color 0 0 0 0)
 	)
 	(junction
@@
 	)
 	(junction
-		(at 120.65 50.8)
-		(diameter 0)
-		(color 0 0 0 0)
-	)
-	(junction
 		(at 134.62 111.76)
 		(diameter 0)
@@
 	(wire
 		(pts
+			(xy 121.92 35.56) (xy 121.92 50.8)
+		)
+		(stroke
+			(width 0)
+			(type default)
+		)
+	)
+	(wire
+		(pts
 			(xy 134.62 121.92) (xy 134.62 111.76)
 		)
@@
 	(wire
 		(pts
+			(xy 121.92 35.56) (xy 132.08 35.56)
+		)
+		(stroke
+			(width 0)
+			(type default)
+		)
+	)
+	(wire
+		(pts
 			(xy 110.49 90.17) (xy 110.49 76.2)
 		)
@@
 	(wire
 		(pts
-			(xy 120.65 33.02) (xy 120.65 50.8)
-		)
-		(stroke
-			(width 0)
-			(type default)
-		)
-	)
-	(wire
-		(pts
 			(xy 144.78 143.51) (xy 142.24 143.51)
 		)
@@
 	(wire
 		(pts
+			(xy 121.92 50.8) (xy 134.62 50.8)
+		)
+		(stroke
+			(width 0)
+			(type default)
+		)
+	)
+	(wire
+		(pts
 			(xy 109.22 50.8) (xy 111.76 50.8)
 		)
@@
 	(wire
 		(pts
-			(xy 120.65 50.8) (xy 134.62 50.8)
+			(xy 119.38 50.8) (xy 121.92 50.8)
 		)
 		(stroke
@@
 	(wire
 		(pts
-			(xy 130.81 35.56) (xy 132.08 35.56)
-		)
-		(stroke
-			(width 0)
-			(type default)
-		)
-	)
-	(wire
-		(pts
 			(xy 146.05 111.76) (xy 149.86 111.76)
 		)
@@
 		(pts
 			(xy 143.51 35.56) (xy 142.24 35.56)
-		)
-		(stroke
-			(width 0)
-			(type default)
-		)
-	)
-	(wire
-		(pts
-			(xy 119.38 50.8) (xy 120.65 50.8)
 		)
 		(stroke
@@
 		(dnp no)
 		(fields_autoplaced yes)
-		(property "Reference" "volume"
+		(property "Reference" "volume1"
 			(at 189.23 82.55 90)
 			(show_name no)
@@
 			(project "Pedal_pcb"
 				(path "/6bb676e9-77fc-434d-95a1-c82abd82b43e"
-					(reference "volume")
+					(reference "volume1")
 					(unit 1)
 				)
@@
 		(dnp no)
 		(fields_autoplaced yes)
-		(property "Reference" "tone"
+		(property "Reference" "tone1"
 			(at 172.72 72.39 90)
 			(show_name no)
@@
 			(project "Pedal_pcb"
 				(path "/6bb676e9-77fc-434d-95a1-c82abd82b43e"
-					(reference "tone")
+					(reference "tone1")
 					(unit 1)
 				)
@@
 		(dnp no)
 		(fields_autoplaced yes)
-		(property "Reference" "gain"
+		(property "Reference" "gain1"
 			(at 142.24 115.57 90)
 			(show_name no)
@@
 			(project "Pedal_pcb"
 				(path "/6bb676e9-77fc-434d-95a1-c82abd82b43e"
-					(reference "gain")
+					(reference "gain1")
 					(unit 1)
 				)
@@
 			)
 		)
-		(property "Footprint" "Package_DFN_QFN:Texas_R-PUQFN-N10"
+		(property "Footprint" ""
 			(at 135.636 35.56 90)
 			(hide yes)
@@
 			)
 		)
-		(property "Footprint" "Package_DFN_QFN:Texas_DSQ0010A_WSON-10-1EP_2x2mm_P0.4mm_EP0.9x1.5mm"
+		(property "Footprint" "Package_DIP:DIP-8_W7.62mm"
 			(at 142.24 78.74 0)
 			(hide yes)
@@
 					(unit 1)
 				)
-			)
-		)
-	)
-	(symbol
-		(lib_id "Switch:SW_SPDT")
-		(at 125.73 33.02 0)
-		(unit 1)
-		(body_style 1)
-		(exclude_from_sim no)
-		(in_bom yes)
-		(on_board yes)
-		(in_pos_files yes)
-		(dnp no)
-		(fields_autoplaced yes)
-		(property "Reference" "SW1"
-			(at 125.73 24.13 0)
-			(show_name no)
-			(do_not_autoplace no)
-			(effects
-				(font
-					(size 1.27 1.27)
-				)
-			)
-		)
-		(property "Value" "SW_SPDT"
-			(at 125.73 26.67 0)
-			(show_name no)
-			(do_not_autoplace no)
-			(effects
-				(font
-					(size 1.27 1.27)
-				)
-			)
-		)
-		(property "Footprint" ""
-			(at 125.73 33.02 0)
-			(hide yes)
-			(show_name no)
-			(do_not_autoplace no)
-			(effects
-				(font
-					(size 1.27 1.27)
-				)
-			)
-		)
-		(property "Datasheet" ""
-			(at 125.73 40.64 0)
-			(hide yes)
-			(show_name no)
-			(do_not_autoplace no)
-			(effects
-				(font
-					(size 1.27 1.27)
-				)
-			)
-		)
-		(property "Description" "Switch, single pole double throw"
-			(at 125.73 33.02 0)
-			(hide yes)
-			(show_name no)
-			(do_not_autoplace no)
-			(effects
-				(font
-					(size 1.27 1.27)
-				)
-			)
-		)
-		(pin "2"
-		)
-		(pin "1"
-		)
-		(pin "3"
-		)
-		(instances
-			(project "Pedal_pcb"
-				(path "/6bb676e9-77fc-434d-95a1-c82abd82b43e"
-					(reference "SW1")
-					(unit 1)
-				)

Commit message: the pcb is done
Parts:
- removed BT1: 9 V, symbol Device:Battery
- removed J1, J2: AudioJack2, symbol Connector_Audio:AudioJack2
- added Battery1, Input1, Output1: Conn_01x02, TestPoint:TestPoint_2Pads_Pitch2.54mm_Drill0.8mm, symbol Connector_Generic:Conn_01x02
Connections:
- net GND: now also Battery1.2 (Pin_2), Input1.2 (Pin_2), Output1.1 (Pin_1)
- net at volume1.2: now also Output1.2 (Pin_2)
- net at R2.1: now also Input1.1 (Pin_1)
- net at C7.1, R4.2: now also Battery1.1 (Pin_1)

Commit message: pcb
Parts:
- added SW1: SW_Nidec_CAS-120A1, Connector_PinHeader_2.54mm:PinHeader_1x03_P2.54mm_Vertical, symbol Switch:SW_Nidec_CAS-120A1
Connections:
- net at Output1.2 (Pin_2), volume1.2: now also SW1.1 (C)
- net at R2.1: now also SW1.3 (A); no longer Input1.1 (Pin_1)
- new net: Input1.1 (Pin_1), SW1.2 (B)
Other:
- note added: "TestPoint:TestPoint_2Pads_Pitch2.54mm_Drill0.8mm"
- moved on the sheet: C4, Output1
Changed lines of the file:
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@@
 	(generator_version "10.0")
 	(paper "A4")
+	(text "TestPoint:TestPoint_2Pads_Pitch2.54mm_Drill0.8mm"
+		(exclude_from_sim no)
+		(at 177.8 43.942 0)
+		(effects
+			(font
+				(size 1.27 1.27)
+			)
+		)
+	)
+	(junction
+		(at 204.47 74.93)
+		(diameter 0)
+		(color 0 0 0 0)
+	)
 	(junction
 		(at 101.6 50.8)
@@
 	(wire
 		(pts
-			(xy 189.23 67.31) (xy 191.77 67.31)
+			(xy 204.47 67.31) (xy 207.01 67.31)
 		)
 		(stroke
@@
 	(wire
 		(pts
-			(xy 189.23 67.31) (xy 189.23 74.93)
+			(xy 204.47 67.31) (xy 204.47 74.93)
 		)
 		(stroke
@@
 	(wire
 		(pts
-			(xy 99.06 90.17) (xy 102.87 90.17)
-		)
-		(stroke
-			(width 0)
-			(type default)
-		)
-	)
-	(wire
-		(pts
 			(xy 138.43 121.92) (xy 134.62 121.92)
 		)
@@
 	(wire
 		(pts
-			(xy 172.72 82.55) (xy 172.72 88.9)
+			(xy 172.72 82.55) (xy 172.72 85.09)
 		)
 		(stroke
@@
 	(wire
 		(pts
-			(xy 193.04 78.74) (xy 198.12 78.74)
+			(xy 193.04 78.74) (xy 196.85 78.74)
 		)
 		(stroke
@@
 	(wire
 		(pts
+			(xy 107.95 106.68) (xy 107.95 100.33)
+		)
+		(stroke
+			(width 0)
+			(type default)
+		)
+	)
+	(wire
+		(pts
 			(xy 125.73 76.2) (xy 134.62 76.2)
 		)
@@
 	(wire
 		(pts
+			(xy 99.06 78.74) (xy 99.06 116.84)
+		)
+		(stroke
+			(width 0)
+			(type default)
+		)
+	)
+	(wire
+		(pts
 			(xy 134.62 92.71) (xy 134.62 101.6)
 		)
@@
 	(wire
 		(pts
+			(xy 107.95 100.33) (xy 204.47 100.33)
+		)
+		(stroke
+			(width 0)
+			(type default)
+		)
+	)
+	(wire
+		(pts
 			(xy 149.86 121.92) (xy 149.86 111.76)
 		)
@@
 	(wire
 		(pts
-			(xy 191.77 62.23) (xy 191.77 64.77)
+			(xy 207.01 62.23) (xy 207.01 64.77)
 		)
 		(stroke
@@
 	(wire
 		(pts
+			(xy 204.47 100.33) (xy 204.47 74.93)
+		)
+		(stroke
+			(width 0)
+			(type default)
+		)
+	)
+	(wire
+		(pts
 			(xy 110.49 76.2) (xy 114.3 76.2)
 		)
@@
 	(wire
 		(pts
-			(xy 99.06 78.74) (xy 99.06 90.17)
-		)
-		(stroke
-			(width 0)
-			(type default)
-		)
-	)
-	(wire
-		(pts
-			(xy 186.69 62.23) (xy 191.77 62.23)
+			(xy 201.93 62.23) (xy 207.01 62.23)
 		)
 		(stroke
@@
 	(wire
 		(pts
+			(xy 99.06 116.84) (xy 105.41 116.84)
+		)
+		(stroke
+			(width 0)
+			(type default)
+		)
+	)
+	(wire
+		(pts
 			(xy 149.86 78.74) (xy 156.21 78.74)
+		)
+		(stroke
+			(width 0)
+			(type default)
+		)
+	)
+	(wire
+		(pts
+			(xy 102.87 90.17) (xy 102.87 106.68)
+		)
+		(stroke
+			(width 0)
+			(type default)
+		)
+	)
+	(wire
+		(pts
+			(xy 204.47 74.93) (xy 189.23 74.93)
 		)
 		(stroke
@@
 	(symbol
 		(lib_id "power:GND")
-		(at 198.12 78.74 0)
+		(at 196.85 78.74 0)
 		(unit 1)
 		(body_style 1)
@@
 		(fields_autoplaced yes)
 		(property "Reference" "#PWR03"
-			(at 198.12 85.09 0)
+			(at 196.85 85.09 0)
 			(hide yes)
 			(show_name no)
@@
 		)
 		(property "Value" "GND"
-			(at 198.12 83.82 0)
+			(at 196.85 83.82 0)
 			(show_name no)
 			(do_not_autoplace no)
@@
 		)
 		(property "Footprint" ""
-			(at 198.12 78.74 0)
+			(at 196.85 78.74 0)
 			(hide yes)
 			(show_name no)
@@
 		)
 		(property "Datasheet" ""
-			(at 198.12 78.74 0)
+			(at 196.85 78.74 0)
 			(hide yes)
 			(show_name no)
@@
 		)
 		(property "Description" "Power symbol creates a global label with name \"GND\" , ground"
-			(at 198.12 78.74 0)
+			(at 196.85 78.74 0)
 			(hide yes)
 			(show_name no)
@@
 	(symbol
 		(lib_id "Device:C")
-		(at 172.72 92.71 0)
+		(at 172.72 88.9 0)
 		(unit 1)
 		(body_style 1)
@@
 		(fields_autoplaced yes)
 		(property "Reference" "C4"
-			(at 176.53 91.4399 0)
+			(at 176.53 87.6299 0)
 			(show_name no)
 			(do_not_autoplace no)
@@
 		)
 		(property "Value" "22 nF"
-			(at 176.53 93.9799 0)
+			(at 176.53 90.1699 0)
 			(show_name no)
 			(do_not_autoplace no)
@@
 		)
 		(property "Footprint" "Capacitor_THT:C_Disc_D3.0mm_W1.6mm_P2.50mm"
-			(at 173.6852 96.52 0)
+			(at 173.6852 92.71 0)
 			(hide yes)
 			(show_name no)
@@
 		)
 		(property "Datasheet" ""
-			(at 172.72 92.71 0)
+			(at 172.72 88.9 0)
 			(hide yes)
 			(show_name no)
@@
 		)
 		(property "Description" "Unpolarized capacitor"
-			(at 172.72 92.71 0)
+			(at 172.72 88.9 0)
 			(hide yes)
 			(show_name no)
@@
 	)
 	(symbol
+		(lib_id "Switch:SW_Nidec_CAS-120A1")
+		(at 105.41 111.76 90)
+		(unit 1)
+		(body_style 1)
+		(exclude_from_sim no)
+		(in_bom yes)
+		(on_board yes)
+		(in_pos_files yes)
+		(dnp no)
+		(fields_autoplaced yes)
+		(property "Reference" "SW1"
+			(at 110.49 110.4899 90)
+			(show_name no)
+			(do_not_autoplace no)
+			(effects
+				(font
+					(size 1.27 1.27)
+				)
+				(justify right)
+			)
+		)
+		(property "Value" "SW_Nidec_CAS-120A1"
+			(at 110.49 113.0299 90)
+			(show_name no)
+			(do_not_autoplace no)
+			(effects
+				(font
+					(size 1.27 1.27)
+				)
+				(justify right)
+			)
+		)
+		(property "Footprint" "Connector_PinHeader_2.54mm:PinHeader_1x03_P2.54mm_Vertical"
+			(at 115.57 111.76 0)
+			(hide yes)
+			(show_name no)
+			(do_not_autoplace no)
+			(effects
+				(font
+					(size 1.27 1.27)
+				)
+			)
+		)
+		(property "Datasheet" "https://www.nidec-components.com/e/catalog/switch/cas.pdf"
+			(at 113.03 111.76 0)
+			(hide yes)
+			(show_name no)
+			(do_not_autoplace no)
+			(effects
+				(font
+					(size 1.27 1.27)
+				)
+			)
+		)
+		(property "Description" "Switch, single pole double throw"
+			(at 105.41 111.76 0)
+			(hide yes)
+			(show_name no)
+			(do_not_autoplace no)
+			(effects
+				(font
+					(size 1.27 1.27)
+				)
+			)
+		)
+		(pin "1"
+		)
+		(pin "2"
+		)
+		(pin "3"
+		)
+		(instances
+			(project "Pedal_pcb"
+				(path "/6bb676e9-77fc-434d-95a1-c82abd82b43e"
+					(reference "SW1")
+					(unit 1)
+				)
+			)
+		)
+	)
+	(symbol
 		(lib_id "Device:C")
 		(at 138.43 143.51 270)
@@
 	(symbol
 		(lib_id "power:GND")
-		(at 186.69 62.23 0)
+		(at 201.93 62.23 0)
 		(unit 1)
 		(body_style 1)
@@
 		(fields_autoplaced yes)
 		(property "Reference" "#PWR04"
-			(at 186.69 68.58 0)
+			(at 201.93 68.58 0)
 			(hide yes)
 			(show_name no)
@@
 		)
 		(property "Value" "GND"
-			(at 186.69 67.31 0)
+			(at 201.93 67.31 0)
 			(show_name no)
 			(do_not_autoplace no)
@@
 		)
 		(property "Footprint" ""
-			(at 186.69 62.23 0)
+			(at 201.93 62.23 0)
 			(hide yes)
 			(show_name no)
@@
 		)
 		(property "Datasheet" ""
-			(at 186.69 62.23 0)
+			(at 201.93 62.23 0)
 			(hide yes)
 			(show_name no)
@@
 		)
 		(property "Description" "Power symbol creates a global label with name \"GND\" , ground"
-			(at 186.69 62.23 0)
+			(at 201.93 62.23 0)
 			(hide yes)
 			(show_name no)
@@
 	(symbol
 		(lib_id "power:GND")
-		(at 172.72 96.52 0)
+		(at 172.72 92.71 0)
 		(unit 1)
 		(body_style 1)
@@
 		(fields_autoplaced yes)
 		(property "Reference" "#PWR02"
-			(at 172.72 102.87 0)
+			(at 172.72 99.06 0)
 			(hide yes)
 			(show_name no)
@@
 		)
 		(property "Value" "GND"
-			(at 172.72 101.6 0)
+			(at 172.72 97.79 0)
 			(show_name no)
 			(do_not_autoplace no)
@@
 		)
 		(property "Footprint" ""
-			(at 172.72 96.52 0)
+			(at 172.72 92.71 0)
 			(hide yes)
 			(show_name no)
@@
 		)
 		(property "Datasheet" ""
-			(at 172.72 96.52 0)
+			(at 172.72 92.71 0)
 			(hide yes)
 			(show_name no)
@@
 		)
 		(property "Description" "Power symbol creates a global label with name \"GND\" , ground"
-			(at 172.72 96.52 0)
+			(at 172.72 92.71 0)
 			(hide yes)
 			(show_name no)
@@
 	(symbol
 		(lib_id "Connector_Generic:Conn_01x02")
-		(at 196.85 64.77 0)
+		(at 212.09 64.77 0)
 		(unit 1)
 		(body_style 1)
@@
 		(fields_autoplaced yes)
 		(property "Reference" "Output1"
-			(at 199.39 64.7699 0)
+			(at 214.63 64.7699 0)
 			(show_name no)
 			(do_not_autoplace no)
@@
 		)
 		(property "Value" "Conn_01x02"
-			(at 199.39 67.3099 0)
+			(at 214.63 67.3099 0)
 			(show_name no)
 			(do_not_autoplace no)
@@
 		)
 		(property "Footprint" "TestPoint:TestPoint_2Pads_Pitch2.54mm_Drill0.8mm"
-			(at 196.85 64.77 0)
+			(at 212.09 64.77 0)
 			(hide yes)
 			(show_name no)
@@
 		)
 		(property "Datasheet" ""
-			(at 196.85 64.77 0)
+			(at 212.09 64.77 0)
 			(hide yes)
 			(show_name no)
@@
 		)
 		(property "Description" "Generic connector, single row, 01x02, script generated (kicad-library-utils/schlib/autogen/connector/)"
-			(at 196.85 64.77 0)
-			(hide yes)
-			(show_name no)
+			(at 212.09 64.77 0)
+			(hide yes)
+			(show_name no)

Commit message: pcb better
Connections:
- net at C7.1, R4.2: now also R2.1, SW1.3 (A); no longer Battery1.1 (Pin_1)
- net at C5.2, R3.1, U1.3 (+): now also Battery1.1 (Pin_1), Input1.1 (Pin_1), SW1.2 (B)
Other:
- note removed: "TestPoint:TestPoint_2Pads_Pitch2.54mm_Drill0.8mm"
- moved on the sheet: Input1
Changed lines of the file:
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@@
 	(generator_version "10.0")
 	(paper "A4")
-	(text "TestPoint:TestPoint_2Pads_Pitch2.54mm_Drill0.8mm"
-		(exclude_from_sim no)
-		(at 177.8 43.942 0)
-		(effects
-			(font
-				(size 1.27 1.27)
-			)
-		)
+	(junction
+		(at 127 50.8)
+		(diameter 0)
+		(color 0 0 0 0)
 	)
 	(junction
@@
 	)
 	(junction
-		(at 121.92 50.8)
+		(at 121.92 76.2)
 		(diameter 0)
 		(color 0 0 0 0)
@@
 	)
 	(junction
+		(at 105.41 116.84)
+		(diameter 0)
+		(color 0 0 0 0)
+	)
+	(junction
 		(at 134.62 121.92)
 		(diameter 0)
@@
 	)
 	(junction
+		(at 102.87 90.17)
+		(diameter 0)
+		(color 0 0 0 0)
+	)
+	(junction
 		(at 134.62 101.6)
 		(diameter 0)
@@
 	(wire
 		(pts
-			(xy 121.92 35.56) (xy 121.92 50.8)
+			(xy 134.62 121.92) (xy 134.62 111.76)
 		)
 		(stroke
@@
 	(wire
 		(pts
-			(xy 134.62 121.92) (xy 134.62 111.76)
+			(xy 146.05 92.71) (xy 149.86 92.71)
 		)
 		(stroke
@@
 	(wire
 		(pts
-			(xy 146.05 92.71) (xy 149.86 92.71)
+			(xy 121.92 35.56) (xy 132.08 35.56)
 		)
 		(stroke
@@
 	(wire
 		(pts
-			(xy 121.92 35.56) (xy 132.08 35.56)
+			(xy 105.41 119.38) (xy 105.41 116.84)
+		)
+		(stroke
+			(width 0)
+			(type default)
+		)
+	)
+	(wire
+		(pts
+			(xy 127 57.15) (xy 127 50.8)
 		)
 		(stroke
@@
 	(wire
 		(pts
-			(xy 99.06 76.2) (xy 101.6 76.2)
+			(xy 97.79 76.2) (xy 100.33 76.2)
 		)
 		(stroke
@@
 	(wire
 		(pts
+			(xy 121.92 35.56) (xy 121.92 76.2)
+		)
+		(stroke
+			(width 0)
+			(type default)
+		)
+	)
+	(wire
+		(pts
 			(xy 138.43 121.92) (xy 134.62 121.92)
 		)
@@
 	(wire
 		(pts
-			(xy 121.92 50.8) (xy 134.62 50.8)
+			(xy 119.38 50.8) (xy 127 50.8)
 		)
 		(stroke
@@
 	(wire
 		(pts
-			(xy 101.6 50.8) (xy 101.6 54.61)
+			(xy 100.33 53.34) (xy 100.33 54.61)
 		)
 		(stroke
@@
 	(wire
 		(pts
-			(xy 99.06 78.74) (xy 99.06 116.84)
+			(xy 97.79 78.74) (xy 97.79 116.84)
 		)
 		(stroke
@@
 	(wire
 		(pts
+			(xy 102.87 90.17) (xy 102.87 57.15)
+		)
+		(stroke
+			(width 0)
+			(type default)
+		)
+	)
+	(wire
+		(pts
 			(xy 149.86 121.92) (xy 149.86 111.76)
 		)
@@
 	(wire
 		(pts
+			(xy 121.92 76.2) (xy 121.92 119.38)
+		)
+		(stroke
+			(width 0)
+			(type default)
+		)
+	)
+	(wire
+		(pts
 			(xy 149.86 92.71) (xy 149.86 78.74)
 		)
@@
 	(wire
 		(pts
-			(xy 119.38 50.8) (xy 121.92 50.8)
+			(xy 121.92 119.38) (xy 105.41 119.38)
+		)
+		(stroke
+			(width 0)
+			(type default)
+		)
+	)
+	(wire
+		(pts
+			(xy 102.87 57.15) (xy 127 57.15)
 		)
 		(stroke
@@
 	(wire
 		(pts
+			(xy 127 50.8) (xy 134.62 50.8)
+		)
+		(stroke
+			(width 0)
+			(type default)
+		)
+	)
+	(wire
+		(pts
 			(xy 146.05 111.76) (xy 149.86 111.76)
 		)
@@
 	(wire
 		(pts
+			(xy 100.33 53.34) (xy 101.6 53.34)
+		)
+		(stroke
+			(width 0)
+			(type default)
+		)
+	)
+	(wire
+		(pts
 			(xy 149.86 111.76) (xy 149.86 101.6)
 		)
@@
 	(wire
 		(pts
-			(xy 99.06 116.84) (xy 105.41 116.84)
+			(xy 97.79 116.84) (xy 105.41 116.84)
+		)
+		(stroke
+			(width 0)
+			(type default)
+		)
+	)
+	(wire
+		(pts
+			(xy 101.6 53.34) (xy 101.6 50.8)
 		)
 		(stroke
@@
 	(symbol
 		(lib_id "power:GND")
-		(at 101.6 76.2 0)
+		(at 100.33 76.2 0)
 		(unit 1)
 		(body_style 1)
@@
 		(fields_autoplaced yes)
 		(property "Reference" "#PWR05"
-			(at 101.6 82.55 0)
+			(at 100.33 82.55 0)
 			(hide yes)
 			(show_name no)
@@
 		)
 		(property "Value" "GND"
-			(at 101.6 81.28 0)
+			(at 100.33 81.28 0)
 			(show_name no)
 			(do_not_autoplace no)
@@
 		)
 		(property "Footprint" ""
-			(at 101.6 76.2 0)
+			(at 100.33 76.2 0)
 			(hide yes)
 			(show_name no)
@@
 		)
 		(property "Datasheet" ""
-			(at 101.6 76.2 0)
+			(at 100.33 76.2 0)
 			(hide yes)
 			(show_name no)
@@
 		)
 		(property "Description" "Power symbol creates a global label with name \"GND\" , ground"
-			(at 101.6 76.2 0)
+			(at 100.33 76.2 0)
 			(hide yes)
 			(show_name no)
@@
 	(symbol
 		(lib_id "power:GND")
-		(at 101.6 54.61 0)
+		(at 100.33 54.61 0)
 		(unit 1)
 		(body_style 1)
@@
 		(fields_autoplaced yes)
 		(property "Reference" "#PWR06"
-			(at 101.6 60.96 0)
+			(at 100.33 60.96 0)
 			(hide yes)
 			(show_name no)
@@
 		)
 		(property "Value" "GND"
-			(at 101.6 59.69 0)
+			(at 100.33 59.69 0)
 			(show_name no)
 			(do_not_autoplace no)
@@
 		)
 		(property "Footprint" ""
-			(at 101.6 54.61 0)
+			(at 100.33 54.61 0)
 			(hide yes)
 			(show_name no)
@@
 		)
 		(property "Datasheet" ""
-			(at 101.6 54.61 0)
+			(at 100.33 54.61 0)
 			(hide yes)
 			(show_name no)
@@
 		)
 		(property "Description" "Power symbol creates a global label with name \"GND\" , ground"
-			(at 101.6 54.61 0)
+			(at 100.33 54.61 0)
 			(hide yes)
 			(show_name no)
@@
 	(symbol
 		(lib_id "Connector_Generic:Conn_01x02")
-		(at 93.98 78.74 180)
+		(at 92.71 78.74 180)
 		(unit 1)
 		(body_style 1)
@@
 		(fields_autoplaced yes)
 		(property "Reference" "Input1"
-			(at 93.98 69.85 0)
+			(at 92.71 69.85 0)
 			(show_name no)
 			(do_not_autoplace no)
@@
 		)
 		(property "Value" "Conn_01x02"
-			(at 93.98 72.39 0)
+			(at 92.71 72.39 0)
 			(show_name no)
 			(do_not_autoplace no)
@@
 		)
 		(property "Footprint" "TestPoint:TestPoint_2Pads_Pitch2.54mm_Drill0.8mm"
-			(at 93.98 78.74 0)
+			(at 92.71 78.74 0)
 			(hide yes)
 			(show_name no)
@@
 		)
 		(property "Datasheet" ""
-			(at 93.98 78.74 0)
+			(at 92.71 78.74 0)
 			(hide yes)
 			(show_name no)
@@
 		)
 		(property "Description" "Generic connector, single row, 01x02, script generated (kicad-library-utils/schlib/autogen/connector/)"
-			(at 93.98 78.74 0)
+			(at 92.71 78.74 0)
 			(hide yes)
 			(show_name no)
